File: Delta sigma.sch (KiCad schematic (older format))
At the start: 12 parts

Commit message: Modify delta sigma for noise shaping with ADC, set analysis goals and analyse up to aliasing
Parts:
- removed C?: 1nF, symbol Device:C
- removed R? (x2): 1.5MΩ, symbol Device:R_US
- removed U? (x2): LM324, symbol Amplifier_Operational:LM324
- added C?: 0.1µF, symbol Device:C_Small
- added C? (x2): 0.1µF, symbol Device:C
- added U?: LM321, Package_TO_SOT_SMD:SOT-23-5, symbol Amplifier_Operational:LM321
- C? (x2): value 1nF -> 100pF
- R?: value 1.5MΩ -> 3.3MΩ
Connections:
- net labels added: ToADC
- net labels removed: Control.Out, Vref
- wire segments 40 -> 43
Other:
- note added: "# Input noise\nFeedback resistor noise and input referred controller current noise directly \nimpact the input SNR. The resistor noise can be made arbitraily small by \nusing a voltage divider and lower resistor value. The controller voltage noise \nonly adds to the ADC noise since it isn’t integrated as the current noise, and\nis thus noise shaped away.\n\n# MOSFET threshold voltage\nMaximum out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"
- note added: "As a rule of thumb, noise shaping of order p and filtering to 1/(2^n) of the \nnyquist bandwidth gives:\n∆SQNR = n · (3 + 6p) dB\nWhereas additional bits of effective resolution give:\n∆SQNR = B · 6.02 dB\nAssuming a common 10-bit ADC with a conservative 8 bits of effective \nresolution, using the first order noise-shaping implemented here and \nequating for 9 additional bits gives:\n9 · 6.02 dB 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"
- note added: "Current"
- note added: "Dimensioning"
- note added: "From measurements, the minimum full scale input current is 1µA. The \nintegration capacitor must be charged up to the full scale ADC voltage with a\nfull scale input current within one period time. Then:\nQ = C · V ⇒ C = I · T / V = I / (V · f) = 1µA / (2V · 2.5kHz) = 800pF"
- note added: "Things to analyse:\n ! Input noise\n ! Find out difference between input referred noise and ADC noise\n ! Find input referred current noise\n ! Find ADC referred noise\n ! MOSFET threshold voltage\n ! Find maximum output voltage from MOSFET threshold voltage\n ! Find whether MOSFET threshold voltage hinders startup\n ! Aliasing?\n ! Find out the effects of aliasing at input\n ! Find out the effec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"
- note added: "This is an integrating differential pulse-code modulation quantiser inspired \nby a delta-sigma ADC and based directly on the lecture ’Sigma-Delta \nModulation’ of the TU Delft EE2S31 course on Signal Processing. See also:\nhttps://cas.tudelft.nl/Education/courses/ee2s31/\n\nTogether with the firmware, the goal of this circuit is to redistribute the ADC\nnoise (both quantisation and otherwise) aw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"
- note added: "Working principle"
- note removed: "(Vcc - Vref) / I_in,max = (3.3V - 1.65V) / 1µA = 1.65MΩ ≈ 1.5MΩ"
- note removed: "Assume input current ~~1µA\nSample rate: 160kHZ for 20 bit resolution\n(1000 steps on oxysignal if it is a 1/1000th of the signal)\n"
- note removed: "Q = C*V ⇒ C ? Q / V = (2 * I_in,max / f_max) / V_max =\n= 2 * 1µA / (160kHz * 1V) = 12.5pF, select 10nF"
- moved on the sheet: C?, Q?, R?
