File: POxiM-wristcomputer.sch (KiCad schematic (older format))
At the start: 25 parts, among them J1 USB_B_Micro, J10 Mains_noise_conn, J11 AudioJack4_Ground, J2 AudioJack4_Ground, J3 USB_B_Micro, J4 USB_A, J5 USB_A, J6 Uart Out, J7 Programming Header, J8 USB_B_Micro, J9 Mains_noise_conn

Commit message: Finalise works-like prototype
Parts:
- J10: value Mains_noise_conn -> Transmissivity in
- J9: value Mains_noise_conn -> Interference in
Changed lines of the file:
@@
 P 7100 5300
 F 0 "J9" H 7028 5538 50  0000 C CNN
-F 1 "Mains_noise_conn" H 7028 5447 50  0000 C CNN
+F 1 "Interference in" H 7028 5447 50  0000 C CNN
 F 2 "Connector_Coaxial:SMA_Molex_73251-2200_Horizontal" H 7100 5300 50  0001 C CNN
 F 3 " ~" H 7100 5300 50  0001 C CNN
@@
 P 7450 5700
 F 0 "J10" H 7378 5938 50  0000 C CNN
-F 1 "Mains_noise_conn" H 7378 5847 50  0000 C CNN
+F 1 "Transmissivity in" H 7378 5847 50  0000 C CNN
 F 2 "Connector_Coaxial:SMA_Molex_73251-2200_Horizontal" H 7450 5700 50  0001 C CNN
 F 3 " ~" H 7450 5700 50  0001 C CNN
@@
 F 5 "517-SJ-5007BK" H 1150 6500 50  0001 C CNN "Order number"
 F 6 "Mouser" H 1150 6500 50  0001 C CNN "Supplier"
-F 7 "" H 1150 6500 50  0001 C CNN "Notes"
-F 8 "https://nl.mouser.com/ProductDetail/3M-Electronic-Specialty/SJ-5007-BLACK?qs=%2Fha2pyFaduiRSYeXVuKtDcQs2AhnnhqqvSF0CPtQzOY%3D" H 1150 6500 50  0001 C CNN "Link"
+F 7 "https://nl.mouser.com/ProductDetail/3M-Electronic-Specialty/SJ-5007-BLACK?qs=%2Fha2pyFaduiRSYeXVuKtDcQs2AhnnhqqvSF0CPtQzOY%3D" H 1150 6500 50  0001 C CNN "Link"
 	1    1150 6500
 	1    0    0    -1
@@
 F 5 "517-SJ-5007BK" H 1150 6750 50  0001 C CNN "Order number"
 F 6 "Mouser" H 1150 6750 50  0001 C CNN "Supplier"
-F 7 "" H 1150 6750 50  0001 C CNN "Notes"
-F 8 "https://nl.mouser.com/ProductDetail/3M-Electronic-Specialty/SJ-5007-BLACK?qs=%2Fha2pyFaduiRSYeXVuKtDcQs2AhnnhqqvSF0CPtQzOY%3D" H 1150 6750 50  0001 C CNN "Link"
+F 7 "https://nl.mouser.com/ProductDetail/3M-Electronic-Specialty/SJ-5007-BLACK?qs=%2Fha2pyFaduiRSYeXVuKtDcQs2AhnnhqqvSF0CPtQzOY%3D" H 1150 6750 50  0001 C CNN "Link"
 	1    1150 6750
 	1    0    0    -1
@@
 F 5 "517-SJ-5007BK" H 1800 6500 50  0001 C CNN "Order number"
 F 6 "Mouser" H 1800 6500 50  0001 C CNN "Supplier"
-F 7 "" H 1800 6500 50  0001 C CNN "Notes"
-F 8 "https://nl.mouser.com/ProductDetail/3M-Electronic-Specialty/SJ-5007-BLACK?qs=%2Fha2pyFaduiRSYeXVuKtDcQs2AhnnhqqvSF0CPtQzOY%3D" H 1800 6500 50  0001 C CNN "Link"
+F 7 "https://nl.mouser.com/ProductDetail/3M-Electronic-Specialty/SJ-5007-BLACK?qs=%2Fha2pyFaduiRSYeXVuKtDcQs2AhnnhqqvSF0CPtQzOY%3D" H 1800 6500 50  0001 C CNN "Link"
 	1    1800 6500
 	1    0    0    -1
@@
 F 5 "517-SJ-5007BK" H 1800 6750 50  0001 C CNN "Order number"
 F 6 "Mouser" H 1800 6750 50  0001 C CNN "Supplier"
-F 7 "" H 1800 6750 50  0001 C CNN "Notes"
-F 8 "https://nl.mouser.com/ProductDetail/3M-Electronic-Specialty/SJ-5007-BLACK?qs=%2Fha2pyFaduiRSYeXVuKtDcQs2AhnnhqqvSF0CPtQzOY%3D" H 1800 6750 50  0001 C CNN "Link"
+F 7 "https://nl.mouser.com/ProductDetail/3M-Electronic-Specialty/SJ-5007-BLACK?qs=%2Fha2pyFaduiRSYeXVuKtDcQs2AhnnhqqvSF0CPtQzOY%3D" H 1800 6750 50  0001 C CNN "Link"
 	1    1800 6750
 	1    0    0    -1
@@
 F 5 "517-SJ-5007BK" H 3350 7250 50  0001 C CNN "Order number"
 F 6 "Mouser" H 3350 7250 50  0001 C CNN "Supplier"
-F 7 "" H 3350 7250 50  0001 C CNN "Notes"
-F 8 "https://nl.mouser.com/ProductDetail/3M-Electronic-Specialty/SJ-5007-BLACK?qs=%2Fha2pyFaduiRSYeXVuKtDcQs2AhnnhqqvSF0CPtQzOY%3D" H 3350 7250 50  0001 C CNN "Link"
+F 7 "https://nl.mouser.com/ProductDetail/3M-Electronic-Specialty/SJ-5007-BLACK?qs=%2Fha2pyFaduiRSYeXVuKtDcQs2AhnnhqqvSF0CPtQzOY%3D" H 3350 7250 50  0001 C CNN "Link"
 	1    3350 7250
 	1    0    0    -1
@@
 F 5 "517-SJ-5007BK" H 3350 7550 50  0001 C CNN "Order number"
 F 6 "Mouser" H 3350 7550 50  0001 C CNN "Supplier"
-F 7 "" H 3350 7550 50  0001 C CNN "Notes"
-F 8 "https://nl.mouser.com/ProductDetail/3M-Electronic-Specialty/SJ-5007-BLACK?qs=%2Fha2pyFaduiRSYeXVuKtDcQs2AhnnhqqvSF0CPtQzOY%3D" H 3350 7550 50  0001 C CNN "Link"
+F 7 "https://nl.mouser.com/ProductDetail/3M-Electronic-Specialty/SJ-5007-BLACK?qs=%2Fha2pyFaduiRSYeXVuKtDcQs2AhnnhqqvSF0CPtQzOY%3D" H 3350 7550 50  0001 C CNN "Link"
 	1    3350 7550
 	1    0    0    -1
@@
 F 5 "517-SJ-5007BK" H 4000 7250 50  0001 C CNN "Order number"
 F 6 "Mouser" H 4000 7250 50  0001 C CNN "Supplier"
-F 7 "" H 4000 7250 50  0001 C CNN "Notes"
-F 8 "https://nl.mouser.com/ProductDetail/3M-Electronic-Specialty/SJ-5007-BLACK?qs=%2Fha2pyFaduiRSYeXVuKtDcQs2AhnnhqqvSF0CPtQzOY%3D" H 4000 7250 50  0001 C CNN "Link"
+F 7 "https://nl.mouser.com/ProductDetail/3M-Electronic-Specialty/SJ-5007-BLACK?qs=%2Fha2pyFaduiRSYeXVuKtDcQs2AhnnhqqvSF0CPtQzOY%3D" H 4000 7250 50  0001 C CNN "Link"
 	1    4000 7250
 	1    0    0    -1
@@
 F 5 "517-SJ-5007BK" H 4000 7550 50  0001 C CNN "Order number"
 F 6 "Mouser" H 4000 7550 50  0001 C CNN "Supplier"
-F 7 "" H 4000 7550 50  0001 C CNN "Notes"
-F 8 "https://nl.mouser.com/ProductDetail/3M-Electronic-Specialty/SJ-5007-BLACK?qs=%2Fha2pyFaduiRSYeXVuKtDcQs2AhnnhqqvSF0CPtQzOY%3D" H 4000 7550 50  0001 C CNN "Link"
+F 7 "https://nl.mouser.com/ProductDetail/3M-Electronic-Specialty/SJ-5007-BLACK?qs=%2Fha2pyFaduiRSYeXVuKtDcQs2AhnnhqqvSF0CPtQzOY%3D" H 4000 7550 50  0001 C CNN "Link"
 	1    4000 7550
 	1    0    0    -1
