File: fake_finger.sch (KiCad schematic (older format))
At the start: 28 parts, among them SW1 Current range, U3 LM358, U4 NLAS4053

Commit message: Finalise works-like prototype
Parts:
- added KN1, KN2: Knob, POxiM-uncategorised:Accesory, symbol POxiM-uncategorised:Accesory
- R10, R8, R9: Link (none) -> https://nl.mouser.com/ProductDetail/Panasonic/ERJ-3EKF2702V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; Order number (none) -> 667-ERJ-3EKF2702V; Part number (none) -> ERJ-3EKF2702V; Supplier (none) -> Mouser
- R11: Link (none) -> https://nl.mouser.com/ProductDetail/Panasonic/ERJ-3EKF1001V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; Order number (none) -> 667-ERJ-3EKF1001V; Part number (none) -> ERJ-3EKF1001V; Supplier (none) -> Mouser
- R12: Link (none) -> https://nl.mouser.com/ProductDetail/Vishay-Dale/CRCW06034M7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; Order number (none) -> 71-CRCW06034M70FKEAC; Part number (none) -> CRCW06034M70FKEAC; Supplier (none) -> Mouser
- R13: Link (none) -> https://nl.mouser.com/ProductDetail/Panasonic/ERJ-3EKF4703V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; Order number (none) -> 667-ERJ-3EKF4703V; Part number (none) -> ERJ-3EKF4703V; Supplier (none) -> Mouser
- R14: Link (none) -> https://nl.mouser.com/ProductDetail/Panasonic/ERJ-3EKF4702V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; Order number (none) -> 667-ERJ-3EKF4702V; Part number (none) -> ERJ-3EKF4702V; Supplier (none) -> Mouser
- R15: Link (none) -> https://nl.mouser.com/ProductDetail/Panasonic/ERJ-3EKF4701V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; Order number (none) -> 667-ERJ-3EKF4701V; Part number (none) -> ERJ-3EKF4701V; Supplier (none) -> Mouser
