File: POxiM-wristcomputer.kicad_pcb (KiCad board)
At the start: 4 copper layers, 42 x 33 mm, 118 parts, among them J1 Power in, J2 To finger probe, Q1 MMBT3904,215, Q2 MMBT3904,215, Q3 MMBT3904,215, Q4 PMBT3906,215, Q5 PMBT3906,215, Q6 PMBT3906,215, Q7 PMBT3906,215, Q8 PMBT3906,215, Q9 PMBT3906,215, U1 LM321, U2 STM8S003F3P, U3 MIC5504-3.3YM5

Commit message: Finish first schematic version
Routing:
- net /USB interface/DataTX: vias 3 -> 2
